Commit message: edit code

File: urdf/Assem3.urdf (robot description, URDF)
Before this commit: robot Assem3, 13 links, 12 joints
Joints:
- joint j11: limit (none) -> lower=-1.70 upper=1.6 effort=10 velocity=3; type continuous -> revolute
- joint j12: type continuous -> fixed
- joint j3: limit (none) -> lower=-2.25 upper=0.9 effort=10 velocity=3; type continuous -> revolute
- joint j4: type continuous -> fixed
- joint j5: limit (none) -> lower=-1.34 upper=1.8 effort=10 velocity=3; type continuous -> revolute
- joint j9: limit (none) -> lower=-1.75 upper=1.6 effort=10 velocity=3; type continuous -> revolute
